Commit message: One lidar setup with right frame names

File: vilma_sensor_kit_description/urdf/sensor_kit.xacro (robot description, xacro)
@@ -20,22 +20,12 @@
     <xacro:property name="calibration" value="${xacro.load_yaml('$(arg config_dir)/sensor_kit_calibration.yaml')}"/>
     <!-- lidar -->
-    <xacro:VLP-16 parent="sensor_kit_base_link" name="velodyne_front" topic="/points_raw" hz="10" samples="220" gpu="$(arg gpu)">
+    <xacro:VLP-16 parent="sensor_kit_base_link" name="vlp16_front" topic="/velodyne_points" hz="10" samples="220" gpu="$(arg gpu)">
       <origin
-        xyz="${calibration['sensor_kit_base_link']['velodyne_front_base_link']['x']}
-             ${calibration['sensor_kit_base_link']['velodyne_front_base_link']['y']}
-             ${calibration['sensor_kit_base_link']['velodyne_front_base_link']['z']}"
-        rpy="${calibration['sensor_kit_base_link']['velodyne_front_base_link']['roll']}
-             ${calibration['sensor_kit_base_link']['velodyne_front_base_link']['pitch']}
-             ${calibration['sensor_kit_base_link']['velodyne_front_base_link']['yaw']}"
-      />
-    </xacro:VLP-16>
-    <xacro:VLP-16 parent="sensor_kit_base_link" name="velodyne_back" topic="/points_raw" hz="10" samples="220" gpu="$(arg gpu)">
-      <origin
-        xyz="${calibration['sensor_kit_base_link']['velodyne_back_base_link']['x']}
-             ${calibration['sensor_kit_base_link']['velodyne_back_base_link']['y']}
-             ${calibration['sensor_kit_base_link']['velodyne_back_base_link']['z']}"
-        rpy="${calibration['sensor_kit_base_link']['velodyne_back_base_link']['roll']}
-             ${calibration['sensor_kit_base_link']['velodyne_back_base_link']['pitch']}
-             ${calibration['sensor_kit_base_link']['velodyne_back_base_link']['yaw']}"
+        xyz="${calibration['sensor_kit_base_link']['vlp16_front']['x']}
+             ${calibration['sensor_kit_base_link']['vlp16_front']['y']}
+             ${calibration['sensor_kit_base_link']['vlp16_front']['z']}"
+        rpy="${calibration['sensor_kit_base_link']['vlp16_front']['roll']}
+             ${calibration['sensor_kit_base_link']['vlp16_front']['pitch']}
+             ${calibration['sensor_kit_base_link']['vlp16_front']['yaw']}"
       />
     </xacro:VLP-16>
@@ -71,13 +61,13 @@
     <!-- imu -->
     <xacro:imu_macro
-      name="tamagawa/imu"
+      name="imu"
       parent="sensor_kit_base_link"
       namespace=""
-      x="${calibration['sensor_kit_base_link']['tamagawa/imu_link']['x']}"
-      y="${calibration['sensor_kit_base_link']['tamagawa/imu_link']['y']}"
-      z="${calibration['sensor_kit_base_link']['tamagawa/imu_link']['z']}"
-      roll="${calibration['sensor_kit_base_link']['tamagawa/imu_link']['roll']}"
-      pitch="${calibration['sensor_kit_base_link']['tamagawa/imu_link']['pitch']}"
-      yaw="${calibration['sensor_kit_base_link']['tamagawa/imu_link']['yaw']}"
+      x="${calibration['sensor_kit_base_link']['imu_link']['x']}"
+      y="${calibration['sensor_kit_base_link']['imu_link']['y']}"
+      z="${calibration['sensor_kit_base_link']['imu_link']['z']}"
+      roll="${calibration['sensor_kit_base_link']['imu_link']['roll']}"
+      pitch="${calibration['sensor_kit_base_link']['imu_link']['pitch']}"
+      yaw="${calibration['sensor_kit_base_link']['imu_link']['yaw']}"
       fps="100"
     />

Commit message: Updating sensor_kit calibration base

File: vilma_sensor_kit_description/urdf/sensor_kit.xacro (robot description, xacro)
@@ -28,4 +28,14 @@
              ${calibration['sensor_kit_base_link']['vlp16_front']['pitch']}
              ${calibration['sensor_kit_base_link']['vlp16_front']['yaw']}"
+      />
+    </xacro:VLP-16>
+    <xacro:VLP-16 parent="sensor_kit_base_link" name="vlp16_back" topic="/velodyne_points" hz="10" samples="220" gpu="$(arg gpu)">
+      <origin
+        xyz="${calibration['sensor_kit_base_link']['vlp16_back']['x']}
+             ${calibration['sensor_kit_base_link']['vlp16_back']['y']}
+             ${calibration['sensor_kit_base_link']['vlp16_back']['z']}"
+        rpy="${calibration['sensor_kit_base_link']['vlp16_back']['roll']}
+             ${calibration['sensor_kit_base_link']['vlp16_back']['pitch']}
+             ${calibration['sensor_kit_base_link']['vlp16_back']['yaw']}"
       />
     </xacro:VLP-16>
